File: Nixie_KiCad/_autosave-Nixie_Clock.kicad_pcb (KiCad board)
At the start: 2 copper layers, 140 x 60 mm, 22 parts, among them U1 K155ID1, U10 K155ID1, U11 IN-14, U12 DS3231, U2 IN-14, U3 K155ID1, U4 IN-14, U5 K155ID1, U6 IN-3, U7 PS_V2H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

Commit message: Finalized Design
- Finalized PCB design
- Generated Gerber files
Other:
- board text added: "github.com/haXoru5/nixie_clock"
Changed lines of the file:
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@@
   (general
     (thickness 1.6)
-    (drawings 5)
+    (drawings 6)
     (tracks 475)
     (zones 0)
@@
   (layers
     (0 F.Cu signal)
-    (31 B.Cu signal hide)
+    (31 B.Cu signal)
     (32 B.Adhes user)
     (33 F.Adhes user)
@@
     (pcbplotparams
       (layerselection 0x010fc_ffffffff)
-      (usegerberextensions false)
-      (usegerberattributes true)
-      (usegerberadvancedattributes true)
-      (creategerberjobfile true)
+      (usegerberextensions true)
+      (usegerberattributes false)
+      (usegerberadvancedattributes false)
+      (creategerberjobfile false)
       (excludeedgelayer true)
       (linewidth 0.100000)
@@
       (psa4output false)
       (plotreference true)
-      (plotvalue true)
+      (plotvalue false)
       (plotinvisibletext false)
       (padsonsilk false)
-      (subtractmaskfromsilk false)
+      (subtractmaskfromsilk true)
       (outputformat 1)
       (mirror false)
-      (drillshape 1)
+      (drillshape 0)
       (scaleselection 1)
-      (outputdirectory ""))
+      (outputdirectory "../Nixie_Gerbers/"))
   )
   (net 0 "")
@@
       (net 7 "Net-(A1-Pad29)"))
   )
-  (gr_text "Nixie Clock V1.0\nMichael Zheng" (at -69.2912 -28.194) (layer F.Cu)
+  (gr_text github.com/haXoru5/nixie_clock (at -60.4012 -28.448) (layer B.SilkS)
+    (effects (font (size 0.7 0.7) (thickness 0.1)) (justify mirror))
+  )
+  (gr_text "Nixie Clock V1.0\nMichael Zheng" (at -69.2912 -28.194) (layer F.SilkS)
     (effects (font (size 0.7 0.7) (thickness 0.1)) (justify left))
   )
